File: hardware/robot.brd (EAGLE design)
At the start: 160 x 100 mm, 91 parts, among them Q1 CSM-3X-CRYSTALCSM-3X, Q2 QRE1113, Q3 QRE1113, Q4 QRE1113, Q5 QRE1113, Q6 CSM-3X-CRYSTALCSM-3X, U1 ATMEGA32U4-AU, U2 ATMEGA32U4-AU, U3 LP2985-33DBVR, U4 MCP1650, U5 MCP73831, X1 05-JST-B5B-XH-A, X2 05-JST-B5B-XH-A

Commit message: new revision
Parts:
- removed AUTO-RESET: SOLDERJUMPERNO, SparkFun:SJ_2S-NO
- removed D1: MBR0520LT, diode:SOD123
- removed JP6: (no value), SparkFun:1X02
- added C22, C23: 18pF, resistor:C1206
- added F1: 1206L, microbuilder:1206_PTC
- added JP1: ISP, SparkFun:2X3
- added L3, RX1, TX1: Green, SparkFun-LED:LED-1206
- added MINIUSB1: MINI-USB-SCHIELD-32005-201, con-cypressindustries:32005-201
- added R20, R21, R22: 1K, resistor:R1206
- added R23, R24: 10K, resistor:R1206
- added R25: 22, resistor:R1206
- added R26, R27: 2.2K, resistor:R1206
- added S1: Reset, SparkFun:TACTILE_SWITCH_SMD
- added SER_CPU2: (no value), pinhead:1X02
- added U$10: PNA460XM, adafruit:PNA460XM
- C1, C10, C12, C13, C14, C15, C16, C2, C3, C4: device sparkfun_2:1206 -> resistor:C1206
- C17: value 18pF -> 1uF; device sparkfun_2:1206 -> resistor:C1206
- C18: value 47U -> 47 µF; device aaron_discrete:C1210K -> resistor:C1206
- C19: device aaron_discrete:R0603-AMR -> resistor:C1206
- C20, C21: device SparkFun:0402-CAP -> resistor:C1206
- C5: value 0.1uF -> 10uF; device sparkfun_2:1206 -> resistor:C1206
- C6: device SparkFun:EIA3216 -> resistor:C1206
- C8: value 18pF -> 0.1uF; device sparkfun_2:1206 -> resistor:C1206
- C9: value 0.1uF -> 1uF; device sparkfun_2:1206 -> resistor:C1206
- D4: device SparkFun:LED-0603 -> SparkFun-LED:LED-1206
- L, RX, TX: device SparkFun:LED-1206 -> SparkFun-LED:LED-1206
- L2: value SDR0403 -> BRL3225T3R3M; device aaron_discrete:SDR0403 -> resistor:L3225P
- R16: value 10K -> 22
- moved C5 471.8 mm to (-77.5, -408.9)
- moved C9 440.9 mm to (-53.3, -379.7)
- moved C2 434.7 mm to (-58.4, -372.1)
- moved U2 373.8 mm to (-72.4, -359.4)
- moved R16 315.0 mm to (-71.1, -408.9)
- moved C17 292.4 mm to (-58.4, -379.7)
- moved C8 292.1 mm to (-77.5, -379.7)
- moved Q6 292.1 mm to (-74.9, -373.4)
- moved C18 50.1 mm to (-77.5, -306.1)
Connections:
- net N$3 renamed XTAL2
- net N$4 renamed XTAL1
- removed net D2/SDA: CONN2.3, CONN3.9, CONN4.9, U1.19
- removed net D3/SCL: CONN2.4, CONN3.10, CONN4.10, U1.18
- removed net LED: U$2.P$8
- removed net MUX5: MUX.5
- removed net MUX6: MUX.2
- removed net MUX7: MUX.4
- removed net RST: AUTO-RESET.1
- removed net S2O5: SHIFT2.4
- removed net S2O6: SHIFT2.5
- removed net S2O7: SHIFT2.6
- removed net S2O8: SHIFT2.7
- removed net SHIFT_SCK: SHIFT1.11, SHIFT2.11
- removed net SHIFT_SER: SHIFT1.14
- removed net VBUS: C5.1, C6.A, D1.A, F2.2
- removed net VCC1: U3.1, U3.3
- removed net VCC2: D3.C, R46.2, R49.2
- removed net VCC_3V3: C11.1, C7.1, U3.5
- removed net VIN: C18.1, CONN5.6, L2.1
- new net 2D+: R16.1, U2.4
- new net 2D-: R25.1, U2.3
- new net 2D13: R20.1, U2.32
- new net 2MISO: JP1.1, U$2.P$11, U$5.P$4, U2.11
- new net 2MOSI: JP1.4, SHIFT1.14, U$2.P$10, U$2.P$6, U$5.P$6, U2.10
- new net 2RESET: JP1.5, R23.1, S1.3, S1.4, U2.13
- new net 2RXLED: R21.1, U2.8
- new net 2SCK: JP1.3, SHIFT1.11, SHIFT2.11, U$2.P$12, U$2.P$7, U$5.P$3, U2.9
- new net 2TXLED: R22.1, U2.22
- new net 2XTAL1: C22.1, Q6.1, U2.17
- new net 2XTAL2: C23.1, Q6.2, U2.16
- new net ECHO: U2.37, ULTRASONIC.2
- new net N$3: SER_CPU2.1, U2.21
- new net N$34: L3.A, R20.2
- new net N$35: R22.2, TX1.C
- new net N$36: R21.2, RX1.C
- new net N$37: MINIUSB1.2, R25.2
- new net N$38: MINIUSB1.3, R16.2
- new net N$4: SER_CPU2.2, U2.20
- new net NRF_CE: U$5.P$2, U2.29
- new net NRF_CSN: U$5.P$7, U2.30
- new net NRF_IRQ: U$5.P$5, U2.1
- new net SCL: CONN2.4, CONN3.10, CONN4.10, R26.1, U$3.P$3, U$4.P$3, U1.18, U2.18
- new net SDA: CONN2.3, CONN3.9, CONN4.9, R27.1, U$3.P$4, U$4.P$4, U1.19, U2.19
- new net SD_CS: U$2.P$9, U2.28
- new net S_GRIP: SERVO2(GRIP).3, U2.27
- new net S_GRIPROT: SERVO3(GRIPROT).3, U2.12
- new net S_USONIC: SERVO1(USONIC).3, U2.31
- new net TFT_CS: U$2.P$3, U2.40
- new net TFT_DC: U$2.P$5, U2.38
- new net TFT_RST: U$2.P$4, U2.39
- new net TRIG: U2.36, ULTRASONIC.3
- new net USB1_VIN: C6.1, D2.1, F2.2
- new net USB2_VIN: C5.1, D2.2, F1.2
- net 3.3V: now also C11.1, C7.1, U$2.P$8, U$5.P$8, U3.5; no longer C3.1, U1.6
- net AREF: now also C8.2, U2.42
- net AVCC: now also U2.24, U2.44
- net GND: now also BATT.2, C18.1, C2.2, C22.2, C23.2, C6.2, C8.1, JP1.6, L3.C, MINIUSB1.5, MINIUSB1.M1, MINIUSB1.M2, MINIUSB1.M3, MINIUSB1.M4, R24.2, S1.1, S1.2, SERVO1(USONIC).1, SERVO2(GRIP).1, SERVO3(GRIPROT).1, U$10.2, U2.15, U2.23, U2.35, U2.43, U2.5, ULTRASONIC.1; no longer C18.2, C6.C, C8.2, JP6.1, R16.2
- net MUX4: now also U$10.1
- net MUX_OUT: now also U2.41
- net N$15: now also C3.1, U1.6; no longer C17.1, Q6.2
- net N$17: now also R24.1, U2.33; no longer C8.1, Q6.1
- net N$18: now also F1.1, MINIUSB1.1; no longer R16.1
- net N$8: now also C9.1, U2.6; no longer AUTO-RESET.2, C2.1
- net RESET: no longer C2.2
- net SHIFT_RCK: now also U2.26
- net USB_VIN: now also D2.3; no longer JP6.2
- net VBATT: now also BATT.1, C18.2, L2.1
- net VCC: now also C17.1, C2.1, D3.C, JP1.2, R23.2, R26.2, R27.2, R46.2, R49.2, RX1.A, SERVO1(USONIC).2, SERVO2(GRIP).2, SERVO3(GRIPROT).2, TX1.A, U$10.3, U2.14, U2.2, U2.34, U2.7, U3.1, U3.3, ULTRASONIC.4; no longer C9.1, D1.C, U$5.P$8

Commit message: new revision
Parts:
- added JP2, JP4: (no value), SparkFun-Connectors:2X3
- CONN1, CONN5: device pinhead:1X06 -> adafruit:1X06-BIG
- CONN2: device pinhead:1X08 -> adafruit:1X08-BIG
- CONN3, CONN4: device pinhead:1X10 -> adafruit:1X10-BIG
- moved R27 491.6 mm to (-86.4, 63.5)
- moved R26 481.4 mm to (-72.4, 58.4)
- moved SER_CPU2 476.4 mm to (-25.4, 38.1)
- moved U$10 457.4 mm to (-87.6, 40.6)
- moved C5 428.1 mm to (-52.1, 18.4)
- moved C22 426.9 mm to (-23.7, 44.6)
- moved C23 426.8 mm to (-18.7, 44.6), turned to 180 degrees
- moved F1 426.1 mm to (-58.4, 18.4)
- moved R25 424.6 mm to (-58.4, 15.6), turned to 180 degrees
- moved R16 422.2 mm to (-58.4, 13.1), turned to 180 degrees
- moved Q6 418.8 mm to (-21.2, 41.9), turned to 180 degrees
- moved MINIUSB1 411.5 mm to (-68.6, 14.0)
- moved U2 389.4 mm to (-21.6, 26.7), turned to 180 degrees
- moved JP1 362.8 mm to (-52.1, 29.2), turned to 270 degrees
- moved C17 362.3 mm to (-74.9, -17.8)
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Connections:
- removed net AGND: FET1.3, Q2.2, Q3.2, Q4.2, Q5.2
- removed net MUX4: MUX.1, U$10.1
- removed net S103: SHIFT1.2, STEPPER_DRIVER.3
- removed net S106: SHIFT1.5, STEPPER_DRIVER.6
- removed net S1O1: SHIFT1.15, STEPPER_DRIVER.1
- removed net S1O2: SHIFT1.1, STEPPER_DRIVER.2
- removed net S1O4: SHIFT1.3, STEPPER_DRIVER.4
- removed net S1O5: SHIFT1.4, STEPPER_DRIVER.5
- removed net S1O7: SHIFT1.6, STEPPER_DRIVER.7
- removed net S1O8: SHIFT1.7, STEPPER_DRIVER.8
- removed net S202: MUX.10, SHIFT2.1
- removed net S2O1: MUX.11, SHIFT2.15
- removed net S2O3: MUX.9, SHIFT2.2
- new net IR: U$10.1, U2.25
- new net IRA: JP4.1, MUX.11
- new net IRB: JP4.3, MUX.10
- new net IRC: JP4.5, MUX.9
- new net IR_GND: JP4.6, MUX.6, MUX.7, MUX.8, Q2.2, Q2.4, Q3.2, Q3.4, Q4.2, Q4.4, Q5.2, Q5.4
- new net IR_OUT: JP4.4, MUX.3
- new net IR_VCC: JP4.2, MUX.16, R1.2, R10.2, R11.2, R12.2, R13.2, R14.2, R15.2, R3.2
- new net N$41: JP2.1, SHIFT2.15
- new net N$42: JP2.3, SHIFT2.1
- new net N$43: JP2.5, SHIFT2.2
- new net N$45: FET1.3, JP2.6
- new net S1: SHIFT1.15, STEPPER_DRIVER.8
- new net S2: SHIFT1.1, STEPPER_DRIVER.7
- new net S3: SHIFT1.2, STEPPER_DRIVER.6
- new net S4: SHIFT1.3, STEPPER_DRIVER.5
- new net S5: SHIFT1.4, STEPPER_DRIVER.4
- new net S6: SHIFT1.5, STEPPER_DRIVER.3
- new net S7: SHIFT1.6, STEPPER_DRIVER.2
- new net S8: SHIFT1.7, STEPPER_DRIVER.1
- net GND: now also BATT.1; no longer BATT.2, MUX.6, MUX.7, MUX.8, Q2.4, Q3.4, Q4.4, Q5.4
- net MUX_OUT: now also JP2.4; no longer MUX.3
- net VBATT: now also BATT.2; no longer BATT.1
- net VCC: now also JP2.2; no longer MUX.16, R1.2, R10.2, R11.2, R12.2, R13.2, R14.2, R15.2, R3.2
Routing:
- net IR_VCC: track 0.00 -> 108.9 mm, vias 0 -> 1
- net VCC: track 0.00 -> 85.9 mm, vias 0 -> 1
- net RESET: track 0.00 -> 75.2 mm, vias 0 -> 4
- net D7: track 0.00 -> 70.4 mm, vias 0 -> 3
- net SDA: track 0.00 -> 67.1 mm, vias 0 -> 1
- net SCL: track 0.00 -> 63.9 mm, vias 0 -> 1
- net IR_GND: track 0.00 -> 55.5 mm
- net AVCC: track 0.00 -> 46.0 mm, vias 0 -> 3
- net MUX2: track 0.00 -> 39.6 mm, vias 0 -> 1
- net D13: track 0.00 -> 38.6 mm
- net D11: track 0.00 -> 38.3 mm, vias 0 -> 1
- net IR_OUT: track 0.00 -> 36.8 mm
- net MUX1: track 0.00 -> 36.7 mm, vias 0 -> 1
- net MUX0: track 0.00 -> 35.6 mm, vias 0 -> 1
- net D6: track 0.00 -> 32.2 mm
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- added copper zone on layer 1, net GND
Other:
- board size 160 x 100 mm -> 276.8 x 194 mm

Commit message: new revision (fuck yeah)
Parts:
- C11: device SparkFun-Passives:0603-CAP -> resistor:C1206
- C7: device SparkFun-Passives:0805 -> resistor:C1206
- moved R18 139.1 mm to (58.4, 20.3)
- moved FET1 138.1 mm to (63.5, 20.3)
- moved D3 92.8 mm to (-52.1, -2.54), turned to 180 degrees
- moved C8 91.0 mm to (-25.7, 16.2), turned to 90 degrees
- moved R46 86.3 mm to (-55.2, -7.94), turned to 90 degrees
- moved C19 84.0 mm to (-61.0, -12.7), turned to 180 degrees
- moved C9 83.5 mm to (-16.5, 25.7)
- moved R24 83.5 mm to (-41.9, 21.0), turned to 180 degrees
- moved R27 83.2 mm to (-3.81, 53.3), turned to 270 degrees
- moved R51 83.1 mm to (-53.0, -12.7), turned to 180 degrees
- moved R17 82.3 mm to (-74.9, -5.08), turned to 180 degrees
- moved R49 80.0 mm to (-51.4, -7.94), turned to 90 degrees
- moved D4 80.0 mm to (-81.3, -5.08)
- moved U5 77.9 mm to (-68.3, -4.13), turned to 90 degrees
- moved R19 77.4 mm to (-74.9, -8.26), turned to 180 degrees
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Connections:
- net USB1_VIN: now also D2.2; no longer D2.1
- net USB2_VIN: now also D2.1; no longer D2.2
Routing:
- net VCC: track 85.9 -> 503.8 mm, vias 1 -> 4
- net TXLED: track 0.00 -> 127.4 mm, vias 0 -> 2
- net RXLED: track 0.00 -> 120.0 mm, vias 0 -> 2
- net 2SCK: track 0.00 -> 116.6 mm, vias 0 -> 6
- net D-: track 2.50 -> 114.0 mm, vias 0 -> 2
- net D+: track 2.65 -> 112.7 mm, vias 0 -> 4
- net S_GRIPROT: track 0.00 -> 104.3 mm, vias 0 -> 1
- net 2MOSI: track 0.00 -> 94.9 mm, vias 0 -> 3
- net N$43: track 0.00 -> 83.1 mm, vias 0 -> 2
- net N$42: track 0.00 -> 78.8 mm, vias 0 -> 1
- net 3.3V: track 0.00 -> 78.5 mm
- net S_GRIP: track 0.00 -> 76.1 mm, vias 0 -> 3
- net N$41: track 0.00 -> 70.7 mm, vias 0 -> 1
- net S2O4: track 0.00 -> 69.1 mm, vias 0 -> 2
- net S_USONIC: track 0.00 -> 66.5 mm, vias 0 -> 1
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- added copper zone on layer 16, net GND
Other:
- outline, holes or cut-outs redrawn

Commit message: final?
Parts:
- moved SER_CPU2 18.2 mm to (-49.5, 41.9), turned to 90 degrees
- moved U$10 15.3 mm to (-64.8, 26.7), turned to 270 degrees
- moved C8 12.3 mm to (-15.9, 8.89), turned to 180 degrees
- moved L3 7.62 mm to (-41.9, 18.4)
- moved R20 7.62 mm to (-41.9, 15.9)
- moved C2 7.62 mm to (-41.9, 10.8)
- moved R24 7.62 mm to (-41.9, 13.3)
- moved U4 2.54 mm to (-58.4, -14.0)
- moved C17 2.54 mm to (-59.4, -5.40)
- moved D3 2.54 mm to (-52.1, 0.00)
- moved FET3 2.54 mm to (-63.5, -4.76)
- moved L2 2.54 mm to (-62.2, -0.64)
- moved R46 2.54 mm to (-55.2, -5.40)
- moved R49 2.54 mm to (-51.4, -5.40)
- moved C19 2.54 mm to (-61.0, -10.2)
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Routing:
- net SHIFT_RCK: track 16.0 -> 132.6 mm, vias 0 -> 6
- net AVCC: track 46.0 -> 159.4 mm, vias 3 -> 9
- net 2MISO: track 31.6 -> 136.6 mm, vias 2 -> 6
- net 2RXLED: track 0.00 -> 86.4 mm, vias 0 -> 2
- net 2MOSI: track 94.9 -> 179.9 mm, vias 3 -> 5
- net 2SCK: track 116.6 -> 194.3 mm, vias 6 -> 9
- net AREF: track 75.8 -> 153.1 mm, vias 2 -> 5
- net VCC: track 503.8 -> 568.9 mm, vias 4 -> 7
- net 2TXLED: track 0.00 -> 63.8 mm, vias 0 -> 2
- net 2D+: track 0.00 -> 56.2 mm, vias 0 -> 2
- net 2D-: track 0.00 -> 54.1 mm, vias 0 -> 2
- net S_USONIC: track 66.5 -> 119.9 mm, vias 1 -> 3
- net NRF_IRQ: track 0.00 -> 50.9 mm, vias 0 -> 2
- net MUX_OUT: track 65.8 -> 111.4 mm
- net S_GRIP: track 76.1 -> 119.0 mm, vias 3 -> 6
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
Commit message: foo
Parts:
- C18: value 47 µF -> 47 uF
- D2: value BAS70-05 -> BAS70
- D4: value Yellow -> POWER
- FET1, FET3: value IRLML2502TR -> TR
- MUX: value 74HC4051_MUX -> 74HC4051
- SERVO1(USONIC): value (none) -> USONIC
- SERVO2(GRIP): value (none) -> GRIPPER
- SERVO3(GRIPROT): value (none) -> ROTATE
- SER_CPU2: value (none) -> SER2
- STEPPER_DRIVER: value (none) -> ULN2803
- U1: value ATMEGA32U4-AU -> USER
- U2: value ATMEGA32U4-AU -> BRAIN
- U3: value LP2985-33DBVR -> LP2985
- moved R11 58.0 mm to (6.99, -25.0)
- moved R13 58.0 mm to (14.6, -25.0)
- moved R15 58.0 mm to (23.5, -25.0)
- moved R3 58.0 mm to (-1.91, -25.0)
- moved MUX 57.6 mm to (10.8, -20.3)
- moved Q2 57.6 mm to (-1.91, -21.6)
- moved Q3 57.6 mm to (6.99, -21.6)
- moved Q4 57.6 mm to (14.6, -21.6)
- moved Q5 57.6 mm to (23.5, -21.6)
- moved R1 57.2 mm to (-1.91, -18.2)
- moved R10 56.7 mm to (6.99, -18.7)
- moved R12 56.7 mm to (14.6, -18.7)
- moved R14 56.7 mm to (23.5, -18.7)
- moved JP4 55.8 mm to (8.26, -13.2)
- moved R8 8.98 mm to (-76.2, 37.5)
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- renumbered L to D13, L3 to D13_2
Routing:
- net VCC: track 568.9 -> 557.3 mm, vias 7 -> 6
- net MUX2: track 40.0 -> 29.3 mm
- net IR_VCC: track 103.3 -> 92.6 mm
- net 2RXLED: track 86.4 -> 77.7 mm
- net 2TXLED: track 63.8 -> 55.4 mm
- net D+: track 112.7 -> 119.1 mm, vias 4 -> 2
- net IR_OUT: track 34.1 -> 27.9 mm, vias 0 -> 1
- net D-: track 114.0 -> 119.0 mm
- net 2D+: track 56.2 -> 51.8 mm
- net USB1_VIN: track 33.9 -> 37.7 mm
- net MUX1: track 34.1 -> 30.7 mm
- net MUX3: track 30.1 -> 27.4 mm
- net IRB: track 8.15 -> 5.66 mm
- net IRA: track 9.23 -> 6.98 mm
- net MUX0: track 30.7 -> 28.9 mm
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Other:
- board size 276.8 x 194 mm -> 156.2 x 103.3 mm
- board text added: "EDUBOT V0.1 BY SEBASTIAN MUSZYTOWSKI"
- board text added: "USER"

Commit message: i can haz gerber
Parts:
- moved C1 91.6 mm to (124.7, 44.5)
- moved C10 91.6 mm to (111.8, 48.3)
- moved C12 91.6 mm to (111.8, 43.2)
- moved C13 91.6 mm to (111.8, 66.0)
- moved C14 91.6 mm to (127.6, 44.5)
- moved C18 91.6 mm to (10.2, 24.8)
- moved C19 91.6 mm to (25.4, 29.2)
- moved C21 91.6 mm to (10.2, 27.9)
- moved C22 91.6 mm to (56.3, 75.1)
- moved C23 91.6 mm to (61.3, 75.1)
- moved C5 91.6 mm to (22.9, 48.9)
- moved CONN1 91.6 mm to (128.3, 33.0)
- moved CONN2 91.6 mm to (125.7, 81.3)
- moved CONN3 91.6 mm to (101.2, 81.3)
- moved CONN5 91.6 mm to (110.5, 33.0)
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