File: hardware/robot.brd (EAGLE design)
At the start: 156.2 x 103.3 mm, 110 parts, among them Q1 CSM-3X-CRYSTALCSM-3X, Q2 QRE1113, Q3 QRE1113, Q4 QRE1113, Q5 QRE1113, Q6 CSM-3X-CRYSTALCSM-3X, U1 USER, U2 BRAIN, U3 LP2985, U4 MCP1650, U5 MCP73831, X1 05-JST-B5B-XH-A, X2 05-JST-B5B-XH-A

Commit message: zeugs
Changed lines of the file:
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@@
 <via x="87.63" y="81.915" extent="1-16" drill="0.3" diameter="0.3048"/>
 <wire x1="87.63" y1="81.915" x2="85.09" y2="81.915" width="0.3048" layer="1"/>
-<wire x1="85.09" y1="81.915" x2="80.3275" y2="77.1525" width="0.3048" layer="1"/>
-<via x="80.3275" y="77.1525" extent="1-16" drill="0.3" diameter="0.3048"/>
-<wire x1="80.3275" y1="77.1525" x2="79.375" y2="76.2" width="0.3048" layer="16"/>
-<wire x1="79.375" y1="76.2" x2="76.2" y2="76.2" width="0.3048" layer="16"/>
-<wire x1="76.2" y1="76.2" x2="68.58" y2="68.58" width="0.3048" layer="16"/>
+<wire x1="85.09" y1="81.915" x2="83.34375" y2="80.16875" width="0.3048" layer="1"/>
 <wire x1="68.58" y1="68.58" x2="62.23" y2="68.58" width="0.3048" layer="16"/>
 <wire x1="62.23" y1="68.58" x2="60.96" y2="67.31" width="0.3048" layer="16"/>
@@
 <wire x1="143.51" y1="78.74" x2="140.6525" y2="78.74" width="0.3048" layer="1"/>
 <wire x1="140.6525" y1="78.74" x2="134.62" y2="84.7725" width="0.3048" layer="1"/>
+<wire x1="83.34375" y1="80.16875" x2="80.01" y2="80.16875" width="0.3048" layer="1"/>
+<wire x1="80.01" y1="80.16875" x2="79.85125" y2="80.01" width="0.3048" layer="1"/>
+<via x="79.85125" y="80.01" extent="1-16" drill="0.3"/>
+<wire x1="79.85125" y1="80.01" x2="79.85125" y2="79.85125" width="0.3048" layer="16"/>
+<wire x1="79.85125" y1="79.85125" x2="68.58" y2="68.58" width="0.3048" layer="16"/>
 </signal>
 <signal name="N$8">

Commit message: zeugs
Parts:
- moved C24 12.4 mm to (27.9, 46.4), turned to 0 degrees
- moved R23 2.83 mm to (38.3, 40.8), turned to 270 degrees
- moved S1 0.32 mm to (36.4, 48.3), turned to 90 degrees
Routing:
- net BATT_OUT: track 35.6 -> 28.8 mm
- net VCC: track 553.5 -> 549.9 mm
- net 2RESET: track 59.3 -> 61.6 mm
- net S_GRIP: track 118.1 -> 119.6 mm
- net GND: vias 130 -> 132
Changed lines of the file:
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@@
 <wire x1="77.47" y1="8.89" x2="77.47" y2="24.13" width="0.3048" layer="20"/>
 <wire x1="77.47" y1="105.41" x2="35.56" y2="105.41" width="0.3048" layer="20"/>
-<text x="8.89" y="90.17" size="1.778" layer="1" font="vector" ratio="21" rot="R180">USER</text>
+<text x="16.51" y="90.17" size="1.778" layer="1" font="vector" ratio="21" rot="R180">USER</text>
 <text x="73.263125" y="97.4725" size="1.778" layer="1" font="vector" ratio="21" rot="R180">EDUBOT V0.12 BY
 SEBASTIAN MUSZYTOWSKI</text>
@@
 <wire x1="79.375" y1="2.06375" x2="114.935" y2="2.06375" width="0.3048" layer="20"/>
 <wire x1="114.935" y1="2.06375" x2="114.935" y2="22.225" width="0.3048" layer="20"/>
+<hole x="3.81" y="90.17" drill="3.2"/>
 </plain>
 <attributes>
@@
 <attribute name="VALUE" x="31.115" y="60.96" size="1.27" layer="27" rot="R270"/>
 </element>
-<element name="R23" library="resistor" package="R1206" value="10K" x="36.5125" y="43.02125" smashed="yes">
-<attribute name="VALUE" x="33.8455" y="41.62425" size="1.27" layer="27" rot="R90"/>
-</element>
-<element name="S1" library="SparkFun" package="TACTILE_SWITCH_SMD" value="Reset" x="36.67125" y="48.26" smashed="yes" rot="R270">
-<attribute name="NAME" x="38.44925" y="49.149" size="0.4064" layer="25" rot="R270"/>
-<attribute name="VALUE" x="34.63925" y="49.149" size="0.4064" layer="27" rot="R270"/>
+<element name="R23" library="resistor" package="R1206" value="10K" x="38.25875" y="40.79875" smashed="yes" rot="R270">
+<attribute name="VALUE" x="39.497" y="37.973" size="1.27" layer="27" rot="R180"/>
+</element>
+<element name="S1" library="SparkFun" package="TACTILE_SWITCH_SMD" value="Reset" x="36.35375" y="48.26" smashed="yes" rot="R90">
+<attribute name="NAME" x="34.57575" y="47.371" size="0.4064" layer="25" rot="R90"/>
+<attribute name="VALUE" x="38.38575" y="47.371" size="0.4064" layer="27" rot="R90"/>
 </element>
 <element name="C2" library="resistor" package="C1206" value="0.1uF" x="44.45" y="41.275" smashed="yes" rot="R180">
@@
 </element>
 <element name="SW1" library="switch" package="SPDT-PTH" value="" x="24.765" y="53.18125" rot="R90"/>
-<element name="C24" library="resistor" package="C1206" value="47 uF" x="27.305" y="33.9725" smashed="yes" rot="R270">
-<attribute name="VALUE" x="28.3845" y="36.5125" size="1.27" layer="27" rot="R270"/>
+<element name="C24" library="resistor" package="C1206" value="47 uF" x="27.94" y="46.355" smashed="yes">
+<attribute name="VALUE" x="25.4" y="47.4345" size="1.27" layer="27"/>
 </element>
 </elements>
@@
 <wire x1="64.22" y1="57.95" x2="72.8725" y2="57.95" width="0.4064" layer="1"/>
 <wire x1="72.8725" y1="57.95" x2="75.8825" y2="60.96" width="0.4064" layer="1"/>
-<wire x1="45.85" y1="39.5" x2="45.85" y2="38.1" width="0.4064" layer="1"/>
+<wire x1="45.85" y1="39.5" x2="45.85" y2="37.205" width="0.4064" layer="1"/>
 <wire x1="45.85" y1="37.205" x2="45.85" y2="34.16" width="0.4064" layer="1"/>
 <wire x1="45.85" y1="34.16" x2="47.87" y2="32.14" width="0.4064" layer="1"/>
@@
 <wire x1="23.94375" y1="54.61" x2="21.59" y2="54.61" width="0.4064" layer="1"/>
 <wire x1="30.48" y1="53.21625" x2="30.48" y2="52.07" width="0.4064" layer="1"/>
-<wire x1="30.48" y1="52.07" x2="30.48" y2="44.29125" width="0.4064" layer="1"/>
-<wire x1="30.48" y1="44.29125" x2="34.44875" y2="40.3225" width="0.4064" layer="1"/>
-<wire x1="34.44875" y1="40.3225" x2="38.1" y2="40.3225" width="0.4064" layer="1"/>
-<wire x1="38.1" y1="40.3225" x2="38.25875" y2="40.3225" width="0.4064" layer="1"/>
-<wire x1="38.25875" y1="40.3225" x2="39.21125" y2="39.37" width="0.4064" layer="1"/>
-<wire x1="39.21125" y1="39.37" x2="41.91" y2="39.37" width="0.4064" layer="1"/>
-<wire x1="37.9345" y1="43.02125" x2="38.1" y2="42.85575" width="0.4064" layer="1"/>
-<wire x1="38.1" y1="42.85575" x2="38.1" y2="40.3225" width="0.4064" layer="1"/>
 <wire x1="45.9075" y1="37.1475" x2="45.85" y2="37.205" width="0.4064" layer="1"/>
-<wire x1="45.85" y1="37.205" x2="45.85" y2="38.1" width="0.4064" layer="1"/>
+<wire x1="38.25875" y1="39.37675" x2="41.90325" y2="39.37675" width="0.4064" layer="1"/>
+<wire x1="41.90325" y1="39.37675" x2="41.91" y2="39.37" width="0.4064" layer="1"/>
+<wire x1="30.48" y1="52.07" x2="30.48" y2="50.8" width="0.4064" layer="1"/>
+<wire x1="30.48" y1="50.8" x2="33.02" y2="48.26" width="0.4064" layer="1"/>
+<wire x1="33.02" y1="48.26" x2="33.02" y2="43.18" width="0.4064" layer="1"/>
+<wire x1="33.02" y1="43.18" x2="36.82325" y2="39.37675" width="0.4064" layer="1"/>
+<wire x1="36.82325" y1="39.37675" x2="38.25875" y2="39.37675" width="0.4064" layer="1"/>
 <wire x1="110.36" y1="48.26" x2="110.36" y2="48.13" width="0" layer="19" extent="1-1"/>
 </signal>
@@
 <via x="68.42125" y="80.645" extent="1-16" drill="0.3" diameter="0.3048"/>
 <via x="65.88125" y="83.185" extent="1-16" drill="0.3" diameter="0.3048"/>
-<via x="76.04125" y="78.105" extent="1-16" drill="0.3" diameter="0.3048"/>
-<via x="76.04125" y="80.645" extent="1-16" drill="0.3" diameter="0.3048"/>
+<via x="70.96125" y="73.025" extent="1-16" drill="0.3" diameter="0.3048"/>
+<via x="70.96125" y="80.645" extent="1-16" drill="0.3" diameter="0.3048"/>
 <via x="73.50125" y="80.645" extent="1-16" drill="0.3" diameter="0.3048"/>
 <via x="51.1175" y="78.58125" extent="1-16" drill="0.3" diameter="0.3048"/>
@@
 <via x="17.78" y="30.48" extent="1-16" drill="0.3" diameter="0.3048"/>
 <via x="28.41625" y="50.8" extent="1-16" drill="0.3" diameter="0.3048"/>
-<via x="28.41625" y="48.26" extent="1-16" drill="0.3" diameter="0.3048"/>
-<via x="32.385" y="49.05375" extent="1-16" drill="0.3" diameter="0.3048"/>
 <via x="32.385" y="51.59375" extent="1-16" drill="0.3" diameter="0.3048"/>
 <via x="71.59625" y="45.72" extent="1-16" drill="0.3" diameter="0.3048"/>
@@
 <via x="53.81625" y="35.56" extent="1-16" drill="0.3" diameter="0.3048"/>
 <via x="110.96625" y="70.32625" extent="1-16" drill="0.3" diameter="0.3048"/>
+<via x="27.6225" y="34.29" extent="1-16" drill="0.3" diameter="0.3048"/>
+<via x="27.6225" y="31.75" extent="1-16" drill="0.3" diameter="0.3048"/>
+<via x="27.6225" y="36.83" extent="1-16" drill="0.3" diameter="0.3048"/>
+<via x="25.0825" y="34.29" extent="1-16" drill="0.3" diameter="0.3048"/>
 </signal>
 <signal name="3.3V">
@@
 <contactref element="S1" pad="4"/>
 <contactref element="U2" pad="13"/>
-<wire x1="34.76625" y1="50.8" x2="34.76625" y2="45.72" width="0.3048" layer="1"/>
+<wire x1="38.25875" y1="45.72" x2="38.25875" y2="50.8" width="0.3048" layer="1"/>
 <wire x1="61.62" y1="62.95" x2="61.62" y2="64.16" width="0.3048" layer="1"/>
 <wire x1="61.62" y1="64.16" x2="62.23" y2="64.77" width="0.3048" layer="1"/>
@@
 <wire x1="39.0525" y1="53.0225" x2="35.8775" y2="53.0225" width="0.3048" layer="16"/>
 <wire x1="35.8775" y1="53.0225" x2="34.29" y2="54.61" width="0.3048" layer="16"/>
-<wire x1="34.76625" y1="50.8" x2="34.76625" y2="54.13375" width="0.4064" layer="1"/>
 <wire x1="34.76625" y1="54.13375" x2="34.29" y2="54.61" width="0.4064" layer="1"/>
-<wire x1="34.76625" y1="45.72" x2="34.76625" y2="43.3455" width="0.4064" layer="1"/>
-<wire x1="34.76625" y1="43.3455" x2="35.0905" y2="43.02125" width="0.4064" layer="1"/>
+<wire x1="34.76625" y1="54.13375" x2="38.1" y2="50.8" width="0.3048" layer="1"/>
+<wire x1="38.1" y1="50.8" x2="38.25875" y2="50.8" width="0.3048" layer="1"/>
+<wire x1="38.25875" y1="45.72" x2="38.1" y2="45.56125" width="0.3048" layer="1"/>
+<wire x1="38.1" y1="45.56125" x2="38.1" y2="42.38625" width="0.4064" layer="1"/>
+<wire x1="38.1" y1="42.38625" x2="38.25875" y2="42.22075" width="0.4064" layer="1"/>
 </signal>
 <signal name="2MOSI">
@@
 <wire x1="143.51" y1="78.74" x2="140.6525" y2="78.74" width="0.3048" layer="1"/>
 <wire x1="140.6525" y1="78.74" x2="134.62" y2="84.7725" width="0.3048" layer="1"/>
-<wire x1="83.34375" y1="80.16875" x2="80.01" y2="80.16875" width="0.3048" layer="1"/>
-<wire x1="80.01" y1="80.16875" x2="79.85125" y2="80.01" width="0.3048" layer="1"/>
-<via x="79.85125" y="80.01" extent="1-16" drill="0.3"/>
-<wire x1="79.85125" y1="80.01" x2="79.85125" y2="79.85125" width="0.3048" layer="16"/>
-<wire x1="79.85125" y1="79.85125" x2="68.58" y2="68.58" width="0.3048" layer="16"/>
+<wire x1="83.34375" y1="80.16875" x2="77.62875" y2="80.16875" width="0.3048" layer="1"/>
+<via x="77.62875" y="80.16875" extent="1-16" drill="0.3"/>
+<wire x1="77.62875" y1="80.16875" x2="75.40625" y2="78.105" width="0.3048" layer="16"/>
+<wire x1="75.40625" y1="78.105" x2="75.40625" y2="75.40625" width="0.3048" layer="16"/>
+<wire x1="75.40625" y1="75.40625" x2="68.58" y2="68.58" width="0.3048" layer="16"/>
 </signal>
 <signal name="N$8">
@@
 <contactref element="C24" pad="1"/>
 <contactref element="SW1" pad="1"/>
-<wire x1="27.305" y1="35.3725" x2="34.925" y2="35.40125" width="0.4064" layer="1"/>
 <wire x1="34.925" y1="35.40125" x2="34.925" y2="35.3945" width="0.4064" layer="1"/>
 <wire x1="26.515" y1="54.68125" x2="26.515" y2="45.5575" width="0.4064" layer="1"/>
@@
 <wire x1="32.22625" y1="40.64" x2="33.29" y2="39.57625" width="0.4064" layer="1"/>
 <wire x1="33.29" y1="39.57625" x2="33.29" y2="38.57" width="0.4064" layer="1"/>
+<wire x1="26.515" y1="45.5575" x2="26.54" y2="46.355" width="0.4064" layer="1"/>
 </signal>
 </signals>
