File: hardware/robot.sch (EAGLE design)
At the start: 91 parts, among them Q1 CSM-3X-CRYSTALCSM-3X, Q2 QRE1113, Q3 QRE1113, Q4 QRE1113, Q5 QRE1113, Q6 CSM-3X-CRYSTALCSM-3X, U1 ATMEGA32U4-AU, U2 ATMEGA32U4-AU, U3 LP2985-33DBVR, U4 MCP1650, U5 MCP73831, X1 05-JST-B5B-XH-A, X2 05-JST-B5B-XH-A

Commit message: new revision
Parts:
- removed AUTO-RESET: SOLDERJUMPERNO, SparkFun:SOLDERJUMPERNO
- removed D1: MBR0520LT, diode:MBR0520LT
- removed JP6: (no value), SparkFun:M02PTH
- added C22, C23: 18pF, resistor:C-EUC1206
- added F1: 1206L, microbuilder:PTC1206_L
- added JP1: ISP, SparkFun:AVR_SPI_PRG_6PTH
- added L3, RX1, TX1: Green, SparkFun-LED:LED1206
- added MINIUSB1: MINI-USB-SCHIELD-32005-201, con-cypressindustries:MINI-USB-SCHIELD-32005-201
- added R20, R21, R22: 1K, resistor:R-EU_R1206
- added R23, R24: 10K, resistor:R-EU_R1206
- added R25: 22, resistor:R-EU_R1206
- added R26, R27: 2.2K, resistor:R-EU_R1206
- added S1: Reset, SparkFun:TAC_SWITCHSMD
- added SER_CPU2: (no value), pinhead:PINHD-1X2
- added U$10: PNA460XM, adafruit:PNA460XM
- C1, C10, C12, C13, C14, C15, C16, C2, C3, C4: device sparkfun_2:CAP1206 -> resistor:C-EUC1206
- C17: value 18pF -> 1uF; device sparkfun_2:CAP1206 -> resistor:C-EUC1206
- C18: value 47U -> 47 µF; device aaron_discrete:CAP_POL1210K -> resistor:C-EUC1206
- C19: device aaron_discrete:C-SMD0603 -> resistor:C-EUC1206
- C20, C21: device SparkFun:CAP0402-CAP -> resistor:C-EUC1206
- C5: value 0.1uF -> 10uF; device sparkfun_2:CAP1206 -> resistor:C-EUC1206
- C6: device SparkFun:CAP_POL1206 -> resistor:C-EUC1206
- C8: value 18pF -> 0.1uF; device sparkfun_2:CAP1206 -> resistor:C-EUC1206
- C9: value 0.1uF -> 1uF; device sparkfun_2:CAP1206 -> resistor:C-EUC1206
- D4: device SparkFun:LED0603 -> SparkFun-LED:LED1206
- L, RX, TX: device SparkFun:LED1206 -> SparkFun-LED:LED1206
- L2: value SDR0403 -> BRL3225T3R3M; device aaron_discrete:SDR0403 -> resistor:L-EUL3225P
- R16: value 10K -> 22
Connections:
- net N$3 renamed XTAL2
- net N$4 renamed XTAL1
- removed net D2/SDA: CONN2.3, CONN3.9, CONN4.9, U1.PD1(INT1/SDA)
- removed net D3/SCL: CONN2.4, CONN3.10, CONN4.10, U1.PD0(INT0/OC0B)
- removed net MUX5: MUX.IO5
- removed net MUX6: MUX.IO6
- removed net MUX7: MUX.IO7
- removed net RST: AUTO-RESET.1
- removed net S2O5: SHIFT2A.QE
- removed net S2O6: SHIFT2A.QF
- removed net S2O7: SHIFT2A.QG
- removed net S2O8: SHIFT2A.QH
- removed net SHIFT_SCK: SHIFT1A.SCK, SHIFT2A.SCK
- removed net SHIFT_SER: SHIFT1A.SER
- removed net VBUS: C5.1, C6.+, D1.A, F2.2
- removed net VCC1: U3.EN, U3.IN
- removed net VCC2: D3.C, R46.2, R49.2
- removed net VCC_3V3: C11.1, C7.1, U3.OUT
- removed net VIN: C18.+, CONN5.6, L2.1
- new net 2D+: R16.1, U2.D+
- new net 2D-: R25.1, U2.D-
- new net 2D13: R20.1, U2.PC7(ICP3/CLK0/OC4A)
- new net 2MISO: JP1.1, U$2.SD_MISO, U$5.MISO, U2.PB3(PDO/MISO)
- new net 2MOSI: JP1.4, SHIFT1A.SER, U$2.SDA, U$2.SD_MOSI, U$5.MOSI, U2.PB2(PDI/MISO)
- new net 2RESET: JP1.5, R23.1, S1.3, S1.4, U2./RESET
- new net 2RXLED: R21.1, U2.PB0(SS)
- new net 2SCK: JP1.3, SHIFT1A.SCK, SHIFT2A.SCK, U$2.SCK, U$2.SD_SCK, U$5.SCK, U2.PB1(SCK)
- new net 2TXLED: R22.1, U2.PD5(XCK/CTS)
- new net 2XTAL1: C22.1, Q6.1, U2.XTAL1
- new net 2XTAL2: C23.1, Q6.2, U2.XTAL2
- new net ECHO: U2.PF6(ADC6/TDO), ULTRASONIC.2
- new net N$3: SER_CPU2.1, U2.PD3(INT3/TXD1)
- new net N$34: L3.A, R20.2
- new net N$35: R22.2, TX1.C
- new net N$36: R21.2, RX1.C
- new net N$37: MINIUSB1G$1.2, R25.2
- new net N$38: MINIUSB1G$1.3, R16.2
- new net N$4: SER_CPU2.2, U2.PD2(INT2/RXD1)
- new net NRF_CE: U$5.CE, U2.PB5(OC1A/OC4B/ADC12)
- new net NRF_CSN: U$5.CSN, U2.PB6(OC1B/OC4B/ADC13)
- new net NRF_IRQ: U$5.IRQ, U2.PE6
- new net SCL: CONN2.4, CONN3.10, CONN4.10, R26.1, U$3.SCL, U$4.SCL, U1.PD0(INT0/OC0B), U2.PD0(INT0/OC0B)
- new net SDA: CONN2.3, CONN3.9, CONN4.9, R27.1, U$3.SDA, U$4.SDA, U1.PD1(INT1/SDA), U2.PD1(INT1/SDA)
- new net SD_CS: U$2.SD_CS, U2.PB4(ADC11)
- new net S_GRIP: SERVO2(GRIP).3, U2.PD7(OC4D/ADC10/T0)
- new net S_GRIPROT: SERVO3(GRIPROT).3, U2.PB7(OC0A/OC1C/RTS)
- new net S_USONIC: SERVO1(USONIC).3, U2.PC6(OC1A)
- new net TFT_CS: U$2.CS, U2.PF1(ADC1)
- new net TFT_DC: U$2.AD, U2.PF5(ADC5/TMS)
- new net TFT_RST: U$2.RESET, U2.PF4(ADC4/TCK)
- new net TRIG: U2.PF7(ADC7(TDI), ULTRASONIC.3
- new net USB1_VIN: C6.1, D2.A1, F2.2
- new net USB2_VIN: C5.1, D2.A2, F1.2
- net 3.3V: now also C11.1, C7.1, U$2.LED, U$5.VCC, U3.OUT; no longer C3.1, U1.UCAP
- net AREF: now also C8.2, U2.AREF
- net AVCC: now also U2.AVCC, U2.AVCC1
- net GND: now also BATT.2, C18.1, C2.2, C22.2, C23.2, C6.2, C8.1, JP1.6, L3.C, MINIUSB1G$1.5, MINIUSB1S.S1, MINIUSB1S.S2, MINIUSB1S.S3, MINIUSB1S.S4, R24.2, S1.1, S1.2, SERVO1(USONIC).1, SERVO2(GRIP).1, SERVO3(GRIPROT).1, SHIFT1P.GND, SHIFT2P.GND, U$10.GND, U$2.GND, U$3.GND, U$4.GND, U$5.GND, U2.GND, U2.GND1, U2.GND2, U2.GND3, U2.UGND, ULTRASONIC.1; no longer C18.-, C6.-, C8.2, JP6.1, R16.2
- net MUX4: now also U$10.OUT
- net MUX_OUT: now also U2.PF0(ADC0)
- net N$15: now also C3.1, U1.UCAP; no longer C17.1, Q6.2
- net N$17: now also R24.1, U2.PE2(HWB); no longer C8.1, Q6.1
- net N$18: now also F1.1, MINIUSB1G$1.1; no longer R16.1
- net N$8: now also C9.1, U2.UCAP; no longer AUTO-RESET.2, C2.1
- net RESET: no longer C2.2
- net SHIFT_RCK: now also U2.PD6(T1/OC4D/ADC9)
- net USB_VIN: now also D2.C; no longer JP6.2
- net VBATT: now also BATT.1, C18.2, L2.1
- net VCC: now also C17.1, C2.1, D3.C, JP1.2, R23.2, R26.2, R27.2, R46.2, R49.2, RX1.A, SERVO1(USONIC).2, SERVO2(GRIP).2, SERVO3(GRIPROT).2, SHIFT1P.VCC, SHIFT2P.VCC, TX1.A, U$10.VCC, U$2.VCC, U$3.VCC, U$4.VCC, U2.UVCC, U2.VBUS, U2.VCC, U2.VCC1, U3.EN, U3.IN, ULTRASONIC.4; no longer C9.1, D1.C
Other:
- note added: "1.8" SPI Display (128*160px)"
- note added: "3.3V LDO"
- note added: "38KHz with digital output"
- note added: "Accelerometer and Gyroscope (GY-521, optional, plug-in module)"
- note added: "Analog Supply (CPU 1 and CPU 2)"
- note added: "CPU 1 (ATMEGA32U4)"
- note added: "CPU 2 (ATMEGA32U4)"
- note added: "Compass (optional, plug-in module)"
- note added: "Edubot V.0.1 by Sebastian Muszytowski <muzy@chaosdorf.de>"
- note added: "GRIP mechanism servo"
- note added: "HC-SR04"
- note added: "HMC5883L"
- note added: "I2C Pullup"
- note added: "IR Reciever"
- note added: "ISP (CPU1)"
- note added: "ISP (CPU2)"
- note added: "LiPo Charge Circuit (PROG = 2K = 500mA)"
- note added: "MPU 6050"
- note added: "NO SUPPORT FOR VIN DUE TO MISSING REGULATOR. EVERYTHING ABOVE 5.5V DAMAGES THE BOARD!"
- note added: "NRF24L01 Breakout"
- note added: "ROTATE mechanism servo"
- note added: "Reset (CPU1)"
- note added: "Reset (CPU2)"
- note added: "Servo 1 (Ultrasonic)"
- note added: "Servo 2 and 3 (Gripper)"
- note added: "Status LEDs (CPU1)"
- note added: "Status LEDs (CPU2)"
- note added: "Step-Up-Converter (2.8 to 4.2Volt to 5V @ 1A)"
- note added: "USB (CPU1)"
- note added: "USB (CPU2)"
- note added: "USB Power Selector"
- note added: "Ultrasonic distance sensor"
- note added: "based on Vinciduino Schematic and ATmega32U4 data sheet; Arduino Leonardo compatible with Headers The user mainly programs this microcontroller."
- note added: "based on Vinciduino Schematic and ATmega32U4 data sheet; Arduino Leonardo compatible without Headers This microcontroller serves as the "brain" interfacing internal components."
- note added: "for moving the Ultrasonic distance sensor to scan the environment"
- note added: "licensed under CC-BY-SA 3.0, based on the beautiful Vinciduino (vinciduino.org), inspired by Sparki (arcbotics.com), made with the lovely Arduino Leonardo in mind (arduino.cc)"
- note added: "on 2x4pin header pinout"
- note added: "optional, only populate when no other component provides pullup resistors! Values may vary (from 2.2K to 10K)"
- note added: "with SD Card Adapter (optional, plug-in module)"
- note removed: "3 to 4.5V IN -> 5V @ 1A OUT"
- note removed: "ATMEGA 32U4"
- note removed: "Analog Supply"
- note removed: "ICSP"
- note removed: "REGULATOR/BOOST"
- note removed: "Reset"
- note removed: "Status LEDs"
- note removed: "USB"
- moved on the sheet: BATT, C1, C10, C11, C12, C13, C14, C15, C16, C17, C2, C20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

Commit message: new revision
Parts:
- added JP2, JP4: (no value), SparkFun-Connectors:M03X22X3_SILK_SM
- CONN1, CONN5: device pinhead:PINHD-1X6 -> adafruit:PINHD-1X6B
- CONN2: device pinhead:PINHD-1X8 -> adafruit:PINHD-1X8BIG
- CONN3, CONN4: device pinhead:PINHD-1X10 -> adafruit:PINHD-1X10
Connections:
- removed net AGND: FET1.D, Q2.K, Q3.K, Q4.K, Q5.K
- removed net MUX4: MUX.IO4, U$10.OUT
- removed net S103: SHIFT1A.QC, STEPPER_DRIVER.3
- removed net S106: SHIFT1A.QF, STEPPER_DRIVER.6
- removed net S1O1: SHIFT1A.QA, STEPPER_DRIVER.1
- removed net S1O2: SHIFT1A.QB, STEPPER_DRIVER.2
- removed net S1O4: SHIFT1A.QD, STEPPER_DRIVER.4
- removed net S1O5: SHIFT1A.QE, STEPPER_DRIVER.5
- removed net S1O7: SHIFT1A.QG, STEPPER_DRIVER.7
- removed net S1O8: SHIFT1A.QH, STEPPER_DRIVER.8
- removed net S202: MUX.B, SHIFT2A.QB
- removed net S2O1: MUX.A, SHIFT2A.QA
- removed net S2O3: MUX.C, SHIFT2A.QC
- new net IR: U$10.OUT, U2.PD4(ICP1/ADC8)
- new net IRA: JP4.1, MUX.A
- new net IRB: JP4.3, MUX.B
- new net IRC: JP4.5, MUX.C
- new net IR_GND: JP4.6, MUX.INH, MUX.VEE, MUX.VSS, Q2.E, Q2.K, Q3.E, Q3.K, Q4.E, Q4.K, Q5.E, Q5.K
- new net IR_OUT: JP4.4, MUX.IO
- new net IR_VCC: JP4.2, MUX.VDD, R1.2, R10.2, R11.2, R12.2, R13.2, R14.2, R15.2, R3.2
- new net N$41: JP2.1, SHIFT2A.QA
- new net N$42: JP2.3, SHIFT2A.QB
- new net N$43: JP2.5, SHIFT2A.QC
- new net N$45: FET1.D, JP2.6
- new net S1: SHIFT1A.QA, STEPPER_DRIVER.8
- new net S2: SHIFT1A.QB, STEPPER_DRIVER.7
- new net S3: SHIFT1A.QC, STEPPER_DRIVER.6
- new net S4: SHIFT1A.QD, STEPPER_DRIVER.5
- new net S5: SHIFT1A.QE, STEPPER_DRIVER.4
- new net S6: SHIFT1A.QF, STEPPER_DRIVER.3
- new net S7: SHIFT1A.QG, STEPPER_DRIVER.2
- new net S8: SHIFT1A.QH, STEPPER_DRIVER.1
- net GND: now also BATT.1; no longer BATT.2, MUX.INH, MUX.VEE, MUX.VSS, Q2.E, Q3.E, Q4.E, Q5.E
- net MUX_OUT: now also JP2.4; no longer MUX.IO
- net VBATT: now also BATT.2; no longer BATT.1
- net VCC: now also JP2.2; no longer MUX.VDD, R1.2, R10.2, R11.2, R12.2, R13.2, R14.2, R15.2, R3.2
Other:
- moved on the sheet: FET1, MUX, Q2, Q3, Q4, Q5, R1, R10, R11, R12, R13, R14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

Commit message: new revision (fuck yeah)
Parts:
- C11: device SparkFun-Passives:CAP0603-CAP -> resistor:C-EUC1206
- C7: device SparkFun-Passives:CAP0805 -> resistor:C-EUC1206
Connections:
- net USB1_VIN: now also D2.A2; no longer D2.A1
- net USB2_VIN: now also D2.A1; no longer D2.A2
Other:
- moved on the sheet: C11, C7
Changed lines of the file:
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@@
 <part name="BATT" library="SparkFun-Connectors" deviceset="M02" device="JST-PTH-VERT"/>
 <part name="GND30" library="SparkFun" deviceset="GND" device=""/>
-<part name="C7" library="SparkFun-Passives" deviceset="CAP" device="0805" value="10uF"/>
+<part name="C7" library="resistor" deviceset="C-EU" device="C1206" value="10uF"/>
 <part name="U3" library="SparkFun" deviceset="V_REG_LDO" device="SMD" value="LP2985-33DBVR"/>
-<part name="C11" library="SparkFun-Passives" deviceset="CAP" device="0603-CAP" value="100nF"/>
+<part name="C11" library="resistor" deviceset="C-EU" device="C1206" value="100nF"/>
 <part name="GND31" library="SparkFun" deviceset="GND" device=""/>
 <part name="Q2" library="aaron_discrete" deviceset="QRE1113" device=""/>
@@
 </segment>
 <segment>
-<wire x1="58.42" y1="134.62" x2="58.42" y2="127" width="0.1524" layer="91"/>
+<wire x1="58.42" y1="132.08" x2="58.42" y2="127" width="0.1524" layer="91"/>
 <pinref part="GND30" gate="1" pin="GND"/>
 <pinref part="C7" gate="G$1" pin="2"/>
 <pinref part="C11" gate="G$1" pin="2"/>
 <wire x1="58.42" y1="127" x2="58.42" y2="124.46" width="0.1524" layer="91"/>
-<wire x1="66.04" y1="134.62" x2="66.04" y2="127" width="0.1524" layer="91"/>
+<wire x1="66.04" y1="132.08" x2="66.04" y2="127" width="0.1524" layer="91"/>
 <wire x1="58.42" y1="127" x2="66.04" y2="127" width="0.1524" layer="91"/>
 <junction x="58.42" y="127"/>
@@
 <segment>
 <pinref part="C7" gate="G$1" pin="1"/>
-<wire x1="58.42" y1="142.24" x2="58.42" y2="147.32" width="0.1524" layer="91"/>
+<wire x1="58.42" y1="139.7" x2="58.42" y2="147.32" width="0.1524" layer="91"/>
 <pinref part="U3" gate="G$1" pin="OUT"/>
 <wire x1="50.8" y1="147.32" x2="58.42" y2="147.32" width="0.1524" layer="91"/>
 <pinref part="C11" gate="G$1" pin="1"/>
 <wire x1="58.42" y1="147.32" x2="66.04" y2="147.32" width="0.1524" layer="91"/>
-<wire x1="66.04" y1="147.32" x2="66.04" y2="142.24" width="0.1524" layer="91"/>
+<wire x1="66.04" y1="147.32" x2="66.04" y2="139.7" width="0.1524" layer="91"/>
 <wire x1="66.04" y1="147.32" x2="73.66" y2="147.32" width="0.1524" layer="91"/>
 <label x="68.58" y="147.32" size="1.778" layer="95"/>
@@
 </segment>
 <segment>
-<pinref part="D2" gate="G$1" pin="A1"/>
-<wire x1="331.47" y1="220.98" x2="327.406" y2="220.98" width="0.1524" layer="91"/>
-<label x="327.66" y="220.98" size="1.778" layer="95" rot="R180" xref="yes"/>
+<pinref part="D2" gate="G$1" pin="A2"/>
+<wire x1="341.63" y1="220.98" x2="356.362" y2="220.98" width="0.1524" layer="91"/>
+<label x="344.424" y="220.98" size="1.778" layer="95"/>
 </segment>
 </net>
@@
 </segment>
 <segment>
-<wire x1="345.44" y1="220.98" x2="341.63" y2="220.98" width="0.1524" layer="91"/>
-<pinref part="D2" gate="G$1" pin="A2"/>
-<label x="345.44" y="220.98" size="1.778" layer="95" xref="yes"/>
-</segment>
-</net>
+<pinref part="D2" gate="G$1" pin="A1"/>
+<wire x1="331.47" y1="220.98" x2="316.992" y2="220.98" width="0.1524" layer="91"/>
+<label x="317.5" y="220.98" size="1.778" layer="95"/>
+</segment>
+</net>

Commit message: foo
Parts:
- C18: value 47 µF -> 47 uF
- D2: value BAS70-05 -> BAS70
- D4: value Yellow -> POWER
- FET1, FET3: value IRLML2502TR -> TR
- MUX: value 74HC4051_MUX -> 74HC4051
- SERVO1(USONIC): value (none) -> USONIC
- SERVO2(GRIP): value (none) -> GRIPPER
- SERVO3(GRIPROT): value (none) -> ROTATE
- SER_CPU2: value (none) -> SER2
- STEPPER_DRIVER: value (none) -> ULN2803
- U1: value ATMEGA32U4-AU -> USER
- U2: value ATMEGA32U4-AU -> BRAIN
- U3: value LP2985-33DBVR -> LP2985
- renumbered L to D13, L3 to D13_2
Changed lines of the file:
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@@
 <part name="GND7" library="SparkFun" deviceset="GND" device=""/>
 <part name="R6" library="resistor" deviceset="R-EU_" device="R1206" value="1K"/>
-<part name="L" library="SparkFun-LED" deviceset="LED" device="1206" value="Green"/>
+<part name="D13" library="SparkFun-LED" deviceset="LED" device="1206" value="Green"/>
 <part name="GND8" library="SparkFun" deviceset="GND" device=""/>
 <part name="GND4" library="SparkFun" deviceset="GND" device=""/>
@@
 <part name="GND13" library="SparkFun" deviceset="GND" device=""/>
 <part name="GND1" library="SparkFun" deviceset="GND" device=""/>
-<part name="U1" library="adafruit" deviceset="ATMEGA32U4" device="-AU"/>
+<part name="U1" library="adafruit" deviceset="ATMEGA32U4" device="-AU" value="USER"/>
 <part name="R7" library="resistor" deviceset="R-EU_" device="R1206" value="1K"/>
 <part name="R8" library="resistor" deviceset="R-EU_" device="R1206" value="1K"/>
@@
 <part name="GND30" library="SparkFun" deviceset="GND" device=""/>
 <part name="C7" library="resistor" deviceset="C-EU" device="C1206" value="10uF"/>
-<part name="U3" library="SparkFun" deviceset="V_REG_LDO" device="SMD" value="LP2985-33DBVR"/>
+<part name="U3" library="SparkFun" deviceset="V_REG_LDO" device="SMD" value="LP2985"/>
 <part name="C11" library="resistor" deviceset="C-EU" device="C1206" value="100nF"/>
 <part name="GND31" library="SparkFun" deviceset="GND" device=""/>
@@
 <part name="R14" library="resistor" deviceset="R-EU_" device="R1206" value="100"/>
 <part name="R15" library="resistor" deviceset="R-EU_" device="R1206" value="10K"/>
-<part name="FET1" library="aaron_discrete" deviceset="IRLML2502TR" device=""/>
+<part name="FET1" library="aaron_discrete" deviceset="IRLML2502TR" device="" value="TR"/>
 <part name="R18" library="resistor" deviceset="R-EU_" device="R1206" value="100"/>
-<part name="MUX" library="SparkFun-AnalogIC" deviceset="74HC4051_MUX" device=""/>
-<part name="STEPPER_DRIVER" library="SparkFun-PowerIC" deviceset="ULN2803" device="SOIC"/>
+<part name="MUX" library="SparkFun-AnalogIC" deviceset="74HC4051_MUX" device="" value="74HC4051"/>
+<part name="STEPPER_DRIVER" library="SparkFun-PowerIC" deviceset="ULN2803" device="SOIC" value="ULN2803"/>
 <part name="U$2" library="muzy_robot" deviceset="1.8TFT+SD" device=""/>
 <part name="U$3" library="muzy_robot" deviceset="GY-521" device=""/>
@@
 <part name="X2" library="con-jst-xh" deviceset="05-JST" device="-B5B-XH-A"/>
 <part name="ULTRASONIC" library="pinhead" deviceset="PINHD-1X4" device=""/>
-<part name="SERVO1(USONIC)" library="pinhead" deviceset="PINHD-1X3" device=""/>
-<part name="SERVO2(GRIP)" library="pinhead" deviceset="PINHD-1X3" device=""/>
-<part name="SERVO3(GRIPROT)" library="pinhead" deviceset="PINHD-1X3" device=""/>
-<part name="D2" library="diode" deviceset="BAS70-05" device=""/>
+<part name="SERVO1(USONIC)" library="pinhead" deviceset="PINHD-1X3" device="" value="USONIC"/>
+<part name="SERVO2(GRIP)" library="pinhead" deviceset="PINHD-1X3" device="" value="GRIPPER"/>
+<part name="SERVO3(GRIPROT)" library="pinhead" deviceset="PINHD-1X3" device="" value="ROTATE"/>
+<part name="D2" library="diode" deviceset="BAS70-05" device="" value="BAS70"/>
 <part name="R49" library="resistor" deviceset="R-EU_" device="R1206" value="3.09k"/>
 <part name="R51" library="resistor" deviceset="R-EU_" device="R1206" value="1K"/>
@@
 <part name="L2" library="resistor" deviceset="L-EU" device="L3225P" value="BRL3225T3R3M"/>
 <part name="D3" library="aaron_discrete" deviceset="B330A" device=""/>
-<part name="FET3" library="aaron_discrete" deviceset="IRLML2502TR" device=""/>
+<part name="FET3" library="aaron_discrete" deviceset="IRLML2502TR" device="" value="TR"/>
 <part name="C20" library="resistor" deviceset="C-EU" device="C1206" value="4.7uF"/>
 <part name="C21" library="resistor" deviceset="C-EU" device="C1206" value="4.7uF"/>
 <part name="GND23" library="supply1" deviceset="GND" device=""/>
 <part name="GND24" library="supply1" deviceset="GND" device=""/>
-<part name="D4" library="SparkFun-LED" deviceset="LED" device="1206" value="Yellow"/>
+<part name="D4" library="SparkFun-LED" deviceset="LED" device="1206" value="POWER"/>
 <part name="R17" library="resistor" deviceset="R-EU_" device="R1206" value="470"/>
 <part name="U5" library="SparkFun" deviceset="MCP73831" device="SMD" value="MCP73831"/>
@@
 <part name="GND38" library="SparkFun" deviceset="GND" device=""/>
 <part name="P+17" library="SparkFun" deviceset="VCC" device=""/>
-<part name="C18" library="resistor" deviceset="C-EU" device="C1206" value="47 µF"/>
+<part name="C18" library="resistor" deviceset="C-EU" device="C1206" value="47 uF"/>
 <part name="GND25" library="supply1" deviceset="GND" device=""/>
 <part name="R20" library="resistor" deviceset="R-EU_" device="R1206" value="1K"/>
-<part name="L3" library="SparkFun-LED" deviceset="LED" device="1206" value="Green"/>
+<part name="D13_2" library="SparkFun-LED" deviceset="LED" device="1206" value="Green"/>
 <part name="GND39" library="SparkFun" deviceset="GND" device=""/>
 <part name="R21" library="resistor" deviceset="R-EU_" device="R1206" value="1K"/>
@@
 <part name="U$9" library="microbuilder" deviceset="AVCC" device=""/>
 <part name="GND42" library="SparkFun" deviceset="GND" device=""/>
-<part name="U2" library="adafruit" deviceset="ATMEGA32U4" device="-AU"/>
+<part name="U2" library="adafruit" deviceset="ATMEGA32U4" device="-AU" value="BRAIN"/>
 <part name="R24" library="resistor" deviceset="R-EU_" device="R1206" value="10K"/>
 <part name="GND43" library="SparkFun" deviceset="GND" device=""/>
@@
 <part name="R27" library="resistor" deviceset="R-EU_" device="R1206" value="2.2K"/>
 <part name="P+3" library="SparkFun" deviceset="VCC" device=""/>
-<part name="SER_CPU2" library="pinhead" deviceset="PINHD-1X2" device=""/>
+<part name="SER_CPU2" library="pinhead" deviceset="PINHD-1X2" device="" value="SER2"/>
 <part name="P+2" library="SparkFun" deviceset="VCC" device=""/>
 <part name="GND49" library="SparkFun" deviceset="GND" device=""/>
@@
 <attribute name="VALUE" x="426.974" y="69.85" size="1.778" layer="96" rot="R90"/>
 </instance>
-<instance part="L" gate="G$1" x="423.672" y="63.5" smashed="yes" rot="MR0">
+<instance part="D13" gate="G$1" x="423.672" y="63.5" smashed="yes" rot="MR0">
 <attribute name="VALUE" x="419.989" y="61.214" size="1.778" layer="96" rot="MR90"/>
 </instance>
@@
 <attribute name="VALUE" x="427.482" y="21.59" size="1.778" layer="96" rot="R90"/>
 </instance>
-<instance part="L3" gate="G$1" x="424.18" y="15.24" smashed="yes" rot="MR0">
+<instance part="D13_2" gate="G$1" x="424.18" y="15.24" smashed="yes" rot="MR0">
 <attribute name="VALUE" x="420.497" y="12.954" size="1.778" layer="96" rot="MR90"/>
 </instance>
@@
 <segment>
 <pinref part="R6" gate="G$1" pin="2"/>
-<pinref part="L" gate="G$1" pin="A"/>
+<pinref part="D13" gate="G$1" pin="A"/>
 </segment>
 </net>
@@
 <segment>
 <wire x1="423.672" y1="55.88" x2="423.672" y2="58.42" width="0.1524" layer="91"/>
-<pinref part="L" gate="G$1" pin="C"/>
+<pinref part="D13" gate="G$1" pin="C"/>
 <pinref part="GND8" gate="1" pin="GND"/>
 </segment>
@@
 <segment>
 <wire x1="424.18" y1="7.62" x2="424.18" y2="10.16" width="0.1524" layer="91"/>
-<pinref part="L3" gate="G$1" pin="C"/>
+<pinref part="D13_2" gate="G$1" pin="C"/>
 <pinref part="GND39" gate="1" pin="GND"/>
 </segment>
@@
 <segment>
 <pinref part="R20" gate="G$1" pin="2"/>
-<pinref part="L3" gate="G$1" pin="A"/>
-</segment>
-</net>
+<pinref part="D13_2" gate="G$1" pin="A"/>
+</segment>
+</net>
