File: hardware/robot.sch (EAGLE design)
At the start: 109 parts, among them Q1 CSM-3X-CRYSTALCSM-3X, Q2 QRE1113, Q3 QRE1113, Q4 QRE1113, Q5 QRE1113, Q6 CSM-3X-CRYSTALCSM-3X, U1 USER, U2 BRAIN, U3 LP2985, U4 MCP1650, U5 MCP73831, X1 05-JST-B5B-XH-A, X2 05-JST-B5B-XH-A

Commit message: foo
Parts:
- removed D2: BAS70, diode:BAS70-05
- added C24: 47 uF, resistor:C-EUC1206
- added SW1: (no value), switch:SPDT
- BATT: value M02JST-PTH-VERT -> M02POLAR_LOCK; device SparkFun-Connectors:M02JST-PTH-VERT -> SparkFun-Connectors:M02POLAR_LOCK
- C19: value 100N -> 0.1uF
- STEPPER_DRIVER: device SparkFun-PowerIC:ULN2803SOIC -> SparkFun-PowerIC:ULN2803SOICW
Connections:
- removed net USB1_VIN: C6.1, D2.A2, F2.2
- removed net USB2_VIN: C5.1, D2.A1, F1.2
- new net BATT_OUT: C24.1, D3.C, R46.2, R49.2, SW1.1
- net GND: now also C24.2
- net USB_VIN: now also C5.1, C6.1, F1.2, F2.2, SW1.3; no longer D2.C
- net VCC: now also SW1.2; no longer D3.C, R46.2, R49.2
Other:
- note added: "Power Selector"
- note removed: "USB Power Selector"
Changed lines of the file:
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@@
 <part name="CONN3" library="adafruit" deviceset="PINHD-1X10" device="" value="DIGITAL"/>
 <part name="CONN4" library="adafruit" deviceset="PINHD-1X10" device="" value="DIGITAL RASTER"/>
-<part name="BATT" library="SparkFun-Connectors" deviceset="M02" device="JST-PTH-VERT"/>
+<part name="BATT" library="SparkFun-Connectors" deviceset="M02" device="POLAR_LOCK" value="M02POLAR_LOCK"/>
 <part name="GND30" library="SparkFun" deviceset="GND" device=""/>
 <part name="C7" library="resistor" deviceset="C-EU" device="C1206" value="10uF"/>
@@
 <part name="R18" library="resistor" deviceset="R-EU_" device="R1206" value="100"/>
 <part name="MUX" library="SparkFun-AnalogIC" deviceset="74HC4051_MUX" device="" value="74HC4051"/>
-<part name="STEPPER_DRIVER" library="SparkFun-PowerIC" deviceset="ULN2803" device="SOIC" value="ULN2803"/>
+<part name="STEPPER_DRIVER" library="SparkFun-PowerIC" deviceset="ULN2803" device="SOICW" value="ULN2803"/>
 <part name="U$2" library="muzy_robot" deviceset="1.8TFT+SD" device=""/>
 <part name="U$3" library="muzy_robot" deviceset="GY-521" device=""/>
@@
 <part name="SERVO2(GRIP)" library="pinhead" deviceset="PINHD-1X3" device="" value="GRIPPER"/>
 <part name="SERVO3(GRIPROT)" library="pinhead" deviceset="PINHD-1X3" device="" value="ROTATE"/>
-<part name="D2" library="diode" deviceset="BAS70-05" device="" value="BAS70"/>
 <part name="R49" library="resistor" deviceset="R-EU_" device="R1206" value="3.09k"/>
 <part name="R51" library="resistor" deviceset="R-EU_" device="R1206" value="1K"/>
 <part name="U4" library="aaron_ic" deviceset="MCP1650" device=""/>
 <part name="R46" library="resistor" deviceset="R-EU_" device="R1206" value="100"/>
-<part name="C19" library="resistor" deviceset="C-EU" device="C1206" value="100N"/>
+<part name="C19" library="resistor" deviceset="C-EU" device="C1206" value="0.1uF"/>
 <part name="L2" library="resistor" deviceset="L-EU" device="L3225P" value="BRL3225T3R3M"/>
 <part name="D3" library="aaron_discrete" deviceset="B330A" device=""/>
@@
 <part name="GND37" library="SparkFun" deviceset="GND" device=""/>
 <part name="GND38" library="SparkFun" deviceset="GND" device=""/>
-<part name="P+17" library="SparkFun" deviceset="VCC" device=""/>
 <part name="C18" library="resistor" deviceset="C-EU" device="C1206" value="47 uF"/>
 <part name="GND25" library="supply1" deviceset="GND" device=""/>
@@
 <part name="P+23" library="SparkFun" deviceset="VCC" device=""/>
 <part name="GND50" library="SparkFun" deviceset="GND" device=""/>
+<part name="SW1" library="switch" deviceset="SPDT" device=""/>
+<part name="C24" library="resistor" deviceset="C-EU" device="C1206" value="47 uF"/>
+<part name="GND33" library="SparkFun" deviceset="GND" device=""/>
+<part name="P+12" library="SparkFun" deviceset="VCC" device=""/>
 </parts>
 <sheets>
@@
 <wire x1="309.88" y1="254" x2="309.88" y2="213.36" width="0.1524" layer="94"/>
 <wire x1="309.88" y1="213.36" x2="363.22" y2="213.36" width="0.1524" layer="94"/>
-<text x="311.15" y="248.666" size="3.81" layer="95" ratio="12">USB Power Selector</text>
+<text x="311.15" y="248.666" size="3.81" layer="95" ratio="12">Power Selector</text>
 <wire x1="363.22" y1="213.36" x2="434.34" y2="213.36" width="0.1524" layer="94"/>
 <wire x1="309.88" y1="254" x2="363.22" y2="254" width="0.1524" layer="94"/>
@@
 <instance part="SERVO2(GRIP)" gate="A" x="353.06" y="302.26"/>
 <instance part="SERVO3(GRIPROT)" gate="A" x="396.24" y="302.26"/>
-<instance part="D2" gate="G$1" x="336.55" y="220.98"/>
 <instance part="R49" gate="G$1" x="256.54" y="30.48" smashed="yes" rot="MR90">
 <attribute name="NAME" x="259.334" y="33.0454" size="1.4224" layer="95" rot="MR180"/>
@@
 <instance part="GND37" gate="1" x="236.22" y="10.16"/>
 <instance part="GND38" gate="1" x="198.12" y="35.56"/>
-<instance part="P+17" gate="1" x="266.7" y="38.1"/>
 <instance part="C18" gate="G$1" x="205.74" y="38.1" smashed="yes" rot="R90">
 <attribute name="NAME" x="208.534" y="45.339" size="1.778" layer="95" rot="R180"/>
@@
 <instance part="P+23" gate="1" x="414.02" y="134.62"/>
 <instance part="GND50" gate="1" x="386.08" y="104.14"/>
+<instance part="SW1" gate="G$1" x="332.74" y="236.22" rot="MR180"/>
+<instance part="C24" gate="G$1" x="269.24" y="35.56" smashed="yes">
+<attribute name="NAME" x="276.479" y="32.766" size="1.778" layer="95" rot="R90"/>
+<attribute name="VALUE" x="273.939" y="32.004" size="1.778" layer="96" rot="R90"/>
+</instance>
+<instance part="GND33" gate="1" x="269.24" y="25.4"/>
+<instance part="P+12" gate="1" x="350.52" y="233.68"/>
 </instances>
 <busses>
@@
 </segment>
 <segment>
-<wire x1="246.38" y1="38.1" x2="256.54" y2="38.1" width="0.1524" layer="91"/>
-<wire x1="256.54" y1="38.1" x2="256.54" y2="35.56" width="0.1524" layer="91"/>
-<wire x1="193.04" y1="43.18" x2="193.04" y2="48.26" width="0.1524" layer="91"/>
-<wire x1="193.04" y1="48.26" x2="256.54" y2="48.26" width="0.1524" layer="91"/>
-<wire x1="256.54" y1="48.26" x2="256.54" y2="38.1" width="0.1524" layer="91"/>
-<wire x1="256.54" y1="38.1" x2="266.7" y2="38.1" width="0.1524" layer="91"/>
-<junction x="256.54" y="38.1"/>
-<pinref part="D3" gate="G$1" pin="C"/>
-<pinref part="R49" gate="G$1" pin="2"/>
-<pinref part="R46" gate="G$1" pin="2"/>
-<pinref part="P+17" gate="1" pin="VCC"/>
-</segment>
-<segment>
 <wire x1="413.004" y1="30.48" x2="413.004" y2="25.4" width="0.1524" layer="91"/>
 <pinref part="P+18" gate="1" pin="VCC"/>
@@
 <pinref part="P+23" gate="1" pin="VCC"/>
 </segment>
+<segment>
+<pinref part="SW1" gate="G$1" pin="2"/>
+<wire x1="337.82" y1="233.68" x2="350.52" y2="233.68" width="0.1524" layer="91"/>
+<pinref part="P+12" gate="1" pin="VCC"/>
+</segment>
 </net>
 <net name="RX-I" class="0">
@@
 <wire x1="386.08" y1="111.76" x2="386.08" y2="106.68" width="0.1524" layer="91"/>
 <pinref part="GND50" gate="1" pin="GND"/>
+</segment>
+<segment>
+<pinref part="C24" gate="G$1" pin="2"/>
+<pinref part="GND33" gate="1" pin="GND"/>
+<wire x1="269.24" y1="27.94" x2="269.24" y2="30.48" width="0.1524" layer="91"/>
 </segment>
 </net>
@@
 </segment>
 <segment>
-<pinref part="D2" gate="G$1" pin="C"/>
-<wire x1="336.55" y1="223.52" x2="336.55" y2="228.346" width="0.1524" layer="91"/>
-<label x="336.55" y="228.346" size="1.778" layer="95" rot="R90" xref="yes"/>
+<pinref part="F1" gate="G$1" pin="2"/>
+<pinref part="C5" gate="G$1" pin="1"/>
+<wire x1="241.3" y1="312.42" x2="241.3" y2="309.88" width="0.1524" layer="91"/>
+<label x="241.3" y="312.42" size="1.778" layer="95" xref="yes"/>
+<wire x1="241.3" y1="309.88" x2="241.3" y2="304.8" width="0.1524" layer="91"/>
+<wire x1="261.62" y1="309.88" x2="241.3" y2="309.88" width="0.1524" layer="91"/>
+</segment>
+<segment>
+<pinref part="F2" gate="G$1" pin="2"/>
+<pinref part="C6" gate="G$1" pin="1"/>
+<wire x1="241.3" y1="256.54" x2="241.3" y2="254" width="0.1524" layer="91"/>
+<label x="241.3" y="256.54" size="1.778" layer="95" xref="yes"/>
+<wire x1="261.62" y1="254" x2="241.3" y2="254" width="0.1524" layer="91"/>
+<wire x1="241.3" y1="254" x2="241.3" y2="248.92" width="0.1524" layer="91"/>
+</segment>
+<segment>
+<pinref part="SW1" gate="G$1" pin="3"/>
+<wire x1="330.2" y1="236.22" x2="317.5" y2="236.22" width="0.1524" layer="91"/>
+<label x="317.5" y="236.22" size="1.778" layer="95"/>
 </segment>
 </net>
@@
 </segment>
 </net>
-<net name="USB1_VIN" class="0">
-<segment>
-<pinref part="F2" gate="G$1" pin="2"/>
-<pinref part="C6" gate="G$1" pin="1"/>
-<wire x1="241.3" y1="256.54" x2="241.3" y2="254" width="0.1524" layer="91"/>
-<label x="241.3" y="256.54" size="1.778" layer="95" xref="yes"/>
-<wire x1="261.62" y1="254" x2="241.3" y2="254" width="0.1524" layer="91"/>
-<wire x1="241.3" y1="254" x2="241.3" y2="248.92" width="0.1524" layer="91"/>
-</segment>
-<segment>
-<pinref part="D2" gate="G$1" pin="A2"/>
-<wire x1="341.63" y1="220.98" x2="356.362" y2="220.98" width="0.1524" layer="91"/>
-<label x="344.424" y="220.98" size="1.778" layer="95"/>
-</segment>
-</net>
 <net name="N$18" class="0">
 <segment>
@@
 <pinref part="MINIUSB1" gate="G$1" pin="3"/>
 <pinref part="R16" gate="G$1" pin="2"/>
-</segment>
-</net>
-<net name="USB2_VIN" class="0">
-<segment>
-<pinref part="F1" gate="G$1" pin="2"/>
-<pinref part="C5" gate="G$1" pin="1"/>
-<wire x1="241.3" y1="312.42" x2="241.3" y2="309.88" width="0.1524" layer="91"/>
-<label x="241.3" y="312.42" size="1.778" layer="95" xref="yes"/>
-<wire x1="241.3" y1="309.88" x2="241.3" y2="304.8" width="0.1524" layer="91"/>
-<wire x1="261.62" y1="309.88" x2="241.3" y2="309.88" width="0.1524" layer="91"/>
-</segment>
-<segment>
-<pinref part="D2" gate="G$1" pin="A1"/>
-<wire x1="331.47" y1="220.98" x2="316.992" y2="220.98" width="0.1524" layer="91"/>
-<label x="317.5" y="220.98" size="1.778" layer="95"/>
 </segment>
 </net>
@@
 </segment>
 </net>
+<net name="BATT_OUT" class="0">
+<segment>
+<wire x1="246.38" y1="38.1" x2="256.54" y2="38.1" width="0.1524" layer="91"/>
+<wire x1="256.54" y1="38.1" x2="256.54" y2="35.56" width="0.1524" layer="91"/>
+<wire x1="193.04" y1="43.18" x2="193.04" y2="48.26" width="0.1524" layer="91"/>
+<wire x1="193.04" y1="48.26" x2="256.54" y2="48.26" width="0.1524" layer="91"/>
+<wire x1="256.54" y1="48.26" x2="256.54" y2="38.1" width="0.1524" layer="91"/>
+<junction x="256.54" y="38.1"/>
+<pinref part="D3" gate="G$1" pin="C"/>
+<pinref part="R49" gate="G$1" pin="2"/>
+<pinref part="R46" gate="G$1" pin="2"/>
+<pinref part="C24" gate="G$1" pin="1"/>
+<wire x1="269.24" y1="38.1" x2="256.54" y2="38.1" width="0.1524" layer="91"/>
+<wire x1="269.24" y1="38.1" x2="269.24" y2="45.72" width="0.1524" layer="91"/>
+<wire x1="269.24" y1="45.72" x2="276.86" y2="45.72" width="0.1524" layer="91"/>
+<label x="269.24" y="45.72" size="1.778" layer="95"/>
+</segment>
+<segment>
+<pinref part="SW1" gate="G$1" pin="1"/>
+<wire x1="330.2" y1="231.14" x2="317.5" y2="231.14" width="0.1524" layer="91"/>
+<label x="317.5" y="231.14" size="1.778" layer="95"/>
+</segment>
+</net>

Commit message: zeugs
Other:
- note added: "Edubot V.0.12 by Sebastian Muszytowski <muzy@muzy.eu>"
- note removed: "Edubot V.0.1 by Sebastian Muszytowski <muzy@chaosdorf.de>"
Changed lines of the file:
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@@
 REGULATOR. EVERYTHING ABOVE 5.5V
 DAMAGES THE BOARD!</text>
-<text x="2.54" y="335.28" size="6.4516" layer="94">Edubot V.0.1 by Sebastian Muszytowski &lt;muzy@chaosdorf.de&gt; </text>
+<text x="2.54" y="335.28" size="6.4516" layer="94">Edubot V.0.12 by Sebastian Muszytowski &lt;muzy@muzy.eu&gt; </text>
 <text x="2.54" y="327.66" size="3.81" layer="94">licensed under CC-BY-SA 3.0, based on the beautiful Vinciduino (vinciduino.org), inspired by Sparki (arcbotics.com), made with the lovely Arduino Leonardo in mind (arduino.cc)</text>
 </plain>
